File: REV Type-C V2.sch (KiCad schematic (older format))
At the start: 22 parts, among them J1 USB_B_Mini, J2 USB_A, J3 USB_C_Receptacle_USB2.0, U1 USB2422, U2 LP2985-3.3, Y1 24M

Commit message: Reorganize and prettify schematic
Parts:
- removed R6, R7: 5.1k, Resistor_SMD:R_0603_1608Metric, symbol Device:R
- added R6, R7: 5.1k, symbol Device:R_Small_US
- C1: symbol Device:C -> Device:C_Small
- C2, C3: value 18p -> 18pF; symbol Device:C -> Device:C_Small
- C4, C5: value 1uf -> 1uF; symbol Device:C -> Device:C_Small
- C6, C7, C8: value 4u7 -> 4.7uF; symbol Device:C -> Device:C_Small
- R1, R2, R4: symbol Device:R -> Device:R_Small_US
- R3, R5: symbol Device:R -> Device:R_US
- U1: symbol Others:USB2422 -> REV-Type-C-V2-rescue:USB2422-Others
- U2: value LP2985-3.3 -> NCP170
Connections:
- net GND: now also C1.1, R6.1, R7.1; no longer C1.2
- net at J3.A5 (CC1): now also R6.2
- net at J3.B5 (CC2): now also R7.2
- net at U1.10 (CRFILT): now also C1.2; no longer C1.1
- net XTALI renamed XTAL_I
- net XTALO renamed XTAL_O
Other:
- note added: "3.3V LDO VREG"
- note added: "Notes:\n1. Omit D1 in place of a better TVS diode arrangement\n2. CC resistors are pulldowns (5.1k) for proper native USB-C operation"
- note added: "USB Crystal"
- note added: "USB Hub"
- note added: "USB Mini-B Output"
- note added: "USB Type-A Output"
- note added: "USB Type-C Input from Phone"
- note added: "to AUX Device"
- note added: "to REV Expansion Hub"
- note removed: "Notes:\n1. Omit D1 in place of a better TVS diode arrangement\n2. CC resistors are pulldowns (5.1k) for proper\n native USB-C operation\n3. LDO is actually NCP170\n"
- moved on the sheet: C1, C2, C3, C4, C5, C6, C7, C8, D1, J1, J2, J3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
