File: REV Type-C V3.sch (KiCad schematic (older format))
At the start: 28 parts, among them J1 USB_B_Mini, J2 USB_A, J3 USB_C_Receptacle_USB2.0, U1 USB2422, U2 MIC5504-3.3YM5, Y1 24M

Commit message: Fix USB hub symbol in schematic
Parts:
- U1: symbol REV-Type-C-V2-rescue:USB2422-Others-REV-Type-C-V2-rescue -> ProjectSpecific:USB2422
Changed lines of the file:
@@
 EESchema Schematic File Version 4
-LIBS:REV Type-C V2-cache
 EELAYER 29 0
 EELAYER END
@@
 $EndComp
 $Comp
-L REV-Type-C-V2-rescue:USB2422-Others-REV-Type-C-V2-rescue U1
+L ProjectSpecific:USB2422 U1
 U 1 1 5CE4110B
 P 1650 4300
